File: hardware/8BitComputer/instruction-register.brd (EAGLE design)
At the start: 100 x 75 mm, 51 parts, among them IC1 SN74LS173ANG4, IC2 SN74LS173ANG4, IC3 SN74LS245NE4, IC4 SN74LS173ANG4, IC5 SN74LS173ANG4, IC6 SN74LS245NE4, J1 BUS OUT, J2 pwr, J4 BUS OUT

Commit message: added holes back
Parts:
- moved J2 10.2 mm to (3.81, 14.0), turned to 270 degrees
Routing:
- net VCC5V: track 284.6 -> 274.5 mm
- net GND: track 243.1 -> 248.8 mm
Changed lines of the file:
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@@
 <layer number="43" name="vRestrict" color="2" fill="10" visible="yes" active="yes"/>
 <layer number="44" name="Drills" color="7" fill="1" visible="no" active="yes"/>
-<layer number="45" name="Holes" color="7" fill="1" visible="no" active="yes"/>
+<layer number="45" name="Holes" color="7" fill="1" visible="yes" active="yes"/>
 <layer number="46" name="Milling" color="3" fill="1" visible="no" active="yes"/>
 <layer number="47" name="Measures" color="7" fill="1" visible="no" active="yes"/>
@@
 <text x="2.54" y="63.5" size="1.016" layer="1">Instruction
 Register</text>
-<text x="88.9" y="3.81" size="1.016" layer="1">Register 3</text>
+<text x="90.17" y="6.35" size="1.016" layer="1">Register 3</text>
+<hole x="2.54" y="72.39" drill="3"/>
+<hole x="97.79" y="72.39" drill="3"/>
+<hole x="97.79" y="2.54" drill="3"/>
+<hole x="2.54" y="2.54" drill="3"/>
 </plain>
 <attributes>
@@
 <attribute name="VALUE" x="11.43" y="31.75" size="1.27" layer="27"/>
 </element>
-<element name="J2" library="connector" package="1X02" value="pwr" x="3.81" y="3.81" smashed="yes">
-<attribute name="NAME" x="2.4638" y="5.6388" size="1.27" layer="25" ratio="10"/>
-<attribute name="VALUE" x="2.54" y="0.635" size="1.27" layer="27"/>
+<element name="J2" library="connector" package="1X02" value="pwr" x="3.81" y="13.97" smashed="yes" rot="R270">
+<attribute name="NAME" x="5.6388" y="15.3162" size="1.27" layer="25" ratio="10" rot="R270"/>
+<attribute name="VALUE" x="0.635" y="15.24" size="1.27" layer="27" rot="R270"/>
 </element>
 <element name="LED1" library="leds" package="LED3MM" value="red" x="72.39" y="3.81" smashed="yes" rot="R270">
@@
 <wire x1="26.024" y1="1.016" x2="24.13" y2="2.91" width="0.4064" layer="1"/>
 <wire x1="29.221" y1="1.016" x2="26.024" y2="1.016" width="0.4064" layer="1"/>
-<wire x1="24.13" y1="2.91" x2="7.25" y2="2.91" width="0.4064" layer="1"/>
-<wire x1="7.25" y1="2.91" x2="6.35" y2="3.81" width="0.4064" layer="1"/>
 <wire x1="65.48133125" y1="73.73874375" x2="65.4025875" y2="73.66" width="0.3048" layer="1"/>
 <wire x1="69.215" y1="72.09" x2="67.56625625" y2="73.73874375" width="0.3048" layer="1"/>
@@
 <wire x1="13.97" y1="53.34" x2="12.7" y2="54.61" width="0.4064" layer="16"/>
 <wire x1="12.7" y1="54.61" x2="12.7" y2="56.04" width="0.4064" layer="16"/>
+<wire x1="3.81" y1="11.43" x2="12.33" y2="2.91" width="0.508" layer="1"/>
+<wire x1="12.33" y1="2.91" x2="24.13" y2="2.91" width="0.508" layer="1"/>
+<wire x1="93.98" y1="56.04" x2="97.409" y2="55.88" width="0" layer="19" extent="1-1"/>
+<wire x1="91.44" y1="56.04" x2="93.98" y2="56.04" width="0" layer="19" extent="1-1"/>
+<wire x1="76.2" y1="56.04" x2="91.44" y2="56.04" width="0" layer="19" extent="1-1"/>
+<wire x1="64.77" y1="56.04" x2="68.834" y2="55.753" width="0" layer="19" extent="1-1"/>
+<wire x1="46.99" y1="56.04" x2="62.23" y2="56.04" width="0" layer="19" extent="1-1"/>
+<wire x1="33.02" y1="56.04" x2="41.275" y2="55.753" width="0" layer="19" extent="1-1"/>
+<wire x1="64.77" y1="36.5" x2="64.77" y2="56.04" width="0" layer="19" extent="1-1"/>
+<wire x1="64.77" y1="17.62" x2="64.77" y2="36.5" width="0" layer="19" extent="1-1"/>
+<wire x1="69.85" y1="17.78" x2="64.77" y2="17.62" width="0" layer="19" extent="1-1"/>
+<wire x1="74.93" y1="17.62" x2="69.85" y2="17.78" width="0" layer="19" extent="1-1"/>
+<wire x1="77.47" y1="17.62" x2="74.93" y2="17.62" width="0" layer="19" extent="1-1"/>
+<wire x1="63.003" y1="2.91" x2="64.77" y2="17.62" width="0" layer="19" extent="1-1"/>
+<wire x1="7.62" y1="17.78" x2="3.81" y2="11.43" width="0" layer="19" extent="1-1"/>
+<wire x1="49.53" y1="17.62" x2="50.049" y2="2.91" width="0" layer="19" extent="1-1"/>
 </signal>
 <signal name="IR_245_OUTPUT_ENABLE">
@@
 <contactref element="C4" pad="2"/>
 <contactref element="J11" pad="4"/>
-<wire x1="3.81" y1="3.81" x2="3.81" y2="21.59" width="0.508" layer="1"/>
 <wire x1="3.81" y1="21.59" x2="7.62" y2="25.4" width="0.508" layer="1"/>
 <wire x1="7.62" y1="25.4" x2="7.78" y2="25.56" width="0.508" layer="1"/>
@@
 <wire x1="93.98" y1="46.228" x2="93.98" y2="48.1" width="0.508" layer="1"/>
 <wire x1="82.347" y1="36.5" x2="90.805" y2="44.958" width="0.508" layer="1"/>
+<wire x1="3.81" y1="13.97" x2="3.81" y2="21.59" width="0.508" layer="1"/>
 </signal>
 <signal name="IR_7">
