File: hardware/8BitComputer/register.brd (EAGLE design)
At the start: 100 x 75 mm, 51 parts, among them IC1 SN74LS173ANG4, IC2 SN74LS173ANG4, IC3 SN74LS245NE4, IC4 SN74LS173ANG4, IC5 SN74LS173ANG4, IC6 SN74LS245NE4, J1 BUS OUT, J2 pwr, J4 BUS OUT

Commit message: added holes back
Parts:
- moved J2 8.89 mm to (3.81, 12.7), turned to 270 degrees
Routing:
- net VCC5V: track 284.6 -> 275.7 mm
- net GND: track 218.8 -> 224.0 mm
Changed lines of the file:
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@@
 <layer number="43" name="vRestrict" color="2" fill="10" visible="yes" active="yes"/>
 <layer number="44" name="Drills" color="7" fill="1" visible="no" active="yes"/>
-<layer number="45" name="Holes" color="7" fill="1" visible="no" active="yes"/>
+<layer number="45" name="Holes" color="7" fill="1" visible="yes" active="yes"/>
 <layer number="46" name="Milling" color="3" fill="1" visible="no" active="yes"/>
 <layer number="47" name="Measures" color="7" fill="1" visible="no" active="yes"/>
@@
 <wire x1="100" y1="75" x2="0" y2="75" width="0" layer="20"/>
 <wire x1="0" y1="75" x2="0" y2="0" width="0" layer="20"/>
+<hole x="2.54" y="72.39" drill="3"/>
+<hole x="97.79" y="72.39" drill="3"/>
+<hole x="97.79" y="2.54" drill="3"/>
+<hole x="2.54" y="2.54" drill="3"/>
 </plain>
 <attributes>
@@
 <attribute name="VALUE" x="11.43" y="31.75" size="1.27" layer="27"/>
 </element>
-<element name="J2" library="connector" package="1X02" value="pwr" x="3.81" y="3.81" smashed="yes">
-<attribute name="NAME" x="2.4638" y="5.6388" size="1.27" layer="25" ratio="10"/>
-<attribute name="VALUE" x="2.54" y="0.635" size="1.27" layer="27"/>
+<element name="J2" library="connector" package="1X02" value="pwr" x="3.81" y="12.7" smashed="yes" rot="R270">
+<attribute name="NAME" x="5.6388" y="14.0462" size="1.27" layer="25" ratio="10" rot="R270"/>
+<attribute name="VALUE" x="0.635" y="13.97" size="1.27" layer="27" rot="R270"/>
 </element>
 <element name="LED1" library="leds" package="LED3MM" value="red" x="72.39" y="3.81" smashed="yes" rot="R270">
@@
 <wire x1="26.024" y1="1.016" x2="24.13" y2="2.91" width="0.4064" layer="1"/>
 <wire x1="29.221" y1="1.016" x2="26.024" y2="1.016" width="0.4064" layer="1"/>
-<wire x1="24.13" y1="2.91" x2="7.25" y2="2.91" width="0.4064" layer="1"/>
-<wire x1="7.25" y1="2.91" x2="6.35" y2="3.81" width="0.4064" layer="1"/>
 <wire x1="65.48133125" y1="73.73874375" x2="65.4025875" y2="73.66" width="0.3048" layer="1"/>
 <wire x1="69.215" y1="72.09" x2="67.56625625" y2="73.73874375" width="0.3048" layer="1"/>
@@
 <wire x1="68.834" y1="55.753" x2="75.913" y2="55.753" width="0.508" layer="1"/>
 <wire x1="75.913" y1="55.753" x2="76.2" y2="56.04" width="0.508" layer="1"/>
+<wire x1="3.81" y1="10.16" x2="11.06" y2="2.91" width="0.508" layer="1"/>
+<wire x1="11.06" y1="2.91" x2="24.13" y2="2.91" width="0.508" layer="1"/>
 </signal>
 <signal name="R1_245_OUTPUT_ENABLE">
@@
 <contactref element="C4" pad="2"/>
 <contactref element="J11" pad="4"/>
-<wire x1="3.81" y1="3.81" x2="3.81" y2="21.59" width="0.508" layer="1"/>
 <wire x1="3.81" y1="21.59" x2="7.62" y2="25.4" width="0.508" layer="1"/>
 <wire x1="7.62" y1="25.4" x2="7.78" y2="25.56" width="0.508" layer="1"/>
@@
 <wire x1="93.98" y1="46.228" x2="93.98" y2="48.1" width="0.508" layer="1"/>
 <wire x1="82.347" y1="36.5" x2="90.805" y2="44.958" width="0.508" layer="1"/>
+<wire x1="3.81" y1="12.7" x2="3.81" y2="21.59" width="0.508" layer="1"/>
 </signal>
 <signal name="R1_173_OUT_B7">
