File: hardware/8BitComputer/clock.sch (EAGLE design)
At the start: 29 parts, among them IC1 LM555CN, J1 Power, J2 Power, J3 CLK_OUTS, Q1 P2N2222AZL1G, Q2 P2N2222AZL1G

Commit message: updated brd
Parts:
- C2: device passives:C-US075-032X103 -> passives:C-USC0805K
- R5: device passives:RESISTORAXIAL-0.3 -> passives:RESISTOR0805-RES
Changed lines of the file:
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@@
 <?xml version="1.0" encoding="utf-8"?>
 <!DOCTYPE eagle SYSTEM "eagle.dtd">
-<eagle version="9.4.0">
+<eagle version="9.5.2">
 <drawing>
 <settings>
@@
 <parts>
 <part name="IC1" library="ICs" deviceset="LM555CN" device=""/>
-<part name="C1" library="passives" deviceset="C-US" device="C0805" value="0.1 uF"/>
+<part name="C1" library="passives" deviceset="C-US" device="C0805" package3d_urn="urn:adsk.eagle:package:8118586/1" value="0.1 uF"/>
 <part name="R1" library="passives" deviceset="RESISTOR" device="0805-RES" value="12 K"/>
 <part name="U$1" library="passives" deviceset="SQUARE-TRIMPOT-POTENTIOMETER" device=""/>
 <part name="R2" library="passives" deviceset="RESISTOR" device="0805-RES" value="1 K"/>
-<part name="C2" library="passives" deviceset="C-US" device="075-032X103" value="100 nF"/>
-<part name="C3" library="passives" deviceset="C-US" device="C0805" value="3.3 uF"/>
+<part name="C2" library="passives" deviceset="C-US" device="C0805K" package3d_urn="urn:adsk.eagle:package:8089589/1" value="100 nF"/>
+<part name="C3" library="passives" deviceset="C-US" device="C0805" package3d_urn="urn:adsk.eagle:package:8118586/1" value="3.3 uF"/>
 <part name="R3" library="passives" deviceset="RESISTOR" device="0805-RES" value="1 K"/>
 <part name="LED1" library="leds" deviceset="LED" device="-3MM-NO_SILK" value="Blue"/>
@@
 <part name="J1" library="connector" deviceset="M02" device="PTH" value="Power"/>
 <part name="U$2" library="switches" deviceset="SWITCH_TACTILE" device="TACTILE_PIN"/>
-<part name="R5" library="passives" deviceset="RESISTOR" device="AXIAL-0.3" value="4.7 K"/>
-<part name="C4" library="passives" deviceset="C-US" device="C0805" value="0.1 uF"/>
+<part name="R5" library="passives" deviceset="RESISTOR" device="0805-RES" value="4.7 K"/>
+<part name="C4" library="passives" deviceset="C-US" device="C0805" package3d_urn="urn:adsk.eagle:package:8118586/1" value="0.1 uF"/>
 <part name="S1" library="switches" deviceset="SWITCH-SPST" device="KIT" value="555 or Manual"/>
-<part name="C5" library="passives" deviceset="C-US" device="C0805" value="0.1 uF"/>
+<part name="C5" library="passives" deviceset="C-US" device="C0805" package3d_urn="urn:adsk.eagle:package:8118586/1" value="0.1 uF"/>
 <part name="LED2" library="leds" deviceset="LED" device="-3MM-NO_SILK" value="Green"/>
 <part name="R6" library="passives" deviceset="RESISTOR" device="0805-RES" value="100 R"/>
@@
 <part name="R8" library="passives" deviceset="RESISTOR" device="0805-RES" value="1 K"/>
 <part name="R9" library="passives" deviceset="RESISTOR" device="0805-RES" value="1 K"/>
-<part name="C6" library="passives" deviceset="C-US" device="C0805" value="0.1 uF"/>
+<part name="C6" library="passives" deviceset="C-US" device="C0805" package3d_urn="urn:adsk.eagle:package:8118586/1" value="0.1 uF"/>
 <part name="J3" library="connector" deviceset="M08" device="SILK_FEMALE_PTH" value="CLK_OUTS"/>
 <part name="J2" library="connector" deviceset="M02" device="PTH" value="Power"/>
@@
 </schematic>
 </drawing>
+<compatibility>
+<note version="8.3" severity="warning">
+Since Version 8.3, EAGLE supports URNs for individual library
+assets (packages, symbols, and devices). The URNs of those assets
+will not be understood (or retained) with this version.
+</note>
+<note version="8.3" severity="warning">
+Since Version 8.3, EAGLE supports the association of 3D packages
+with devices in libraries, schematics, and board files. Those 3D
+packages will not be understood (or retained) with this version.
+</note>
+</compatibility>
 </eagle>
